File: STM32-FOC-hardware/ESC-BLDC/ESC-BLDC.kicad_sch (KiCad schematic)
At the start: 10 parts, among them P7 JST_SH-02P, P8 JST_SH-02P, U4 MCP2551-I/SN

Commit message: Exclude unresolved JST connectors from assembly
Parts:
- P7, P8: DNP (none) -> Yes; LCSC C160402 -> (none); MPN SM02B-SRSS-TB(LF)(SN) -> (none); now not fitted; now left out of the parts list
Changed lines of the file:
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@@
 		(body_style 1)
 		(exclude_from_sim no)
-		(in_bom yes)
+		(in_bom no)
 		(on_board yes)
-		(in_pos_files yes)
-		(dnp no)
-		(property "LCSC" "C160402"
+		(in_pos_files no)
+		(dnp yes)
+		(property "DNP" "Yes"
 			(at 177.8 143.9672 0)
 			(hide yes)
@@
 			(effects (font (size 1.27 1.27)))
 		)
-		(property "MPN" "SM02B-SRSS-TB(LF)(SN)"
+		(property "LCSC" ""
+			(at 177.8 143.9672 0)
+			(hide yes)
+			(show_name no)
+			(do_not_autoplace no)
+			(effects (font (size 1.27 1.27)))
+		)
+		(property "MPN" ""
 			(at 177.8 143.9672 0)
 			(hide yes)
@@
 		(body_style 1)
 		(exclude_from_sim no)
-		(in_bom yes)
+		(in_bom no)
 		(on_board yes)
-		(in_pos_files yes)
-		(dnp no)
-		(property "LCSC" "C160402"
+		(in_pos_files no)
+		(dnp yes)
+		(property "DNP" "Yes"
 			(at 177.8 128.7272 0)
 			(hide yes)
@@
 			(effects (font (size 1.27 1.27)))
 		)
-		(property "MPN" "SM02B-SRSS-TB(LF)(SN)"
+		(property "LCSC" ""
 			(at 177.8 128.7272 0)
 			(hide yes)
+			(show_name no)
+			(do_not_autoplace no)
+			(effects (font (size 1.27 1.27)))
+		)
+		(property "MPN" ""
+			(at 177.8 128.7272 0)
+			(hide yes)

Commit message: Apply schematic cleanup and sourcing todo
Parts:
- P7, P8: value JST_SH-02P -> SM02B-SRSS-TB; MPN (none) -> SM02B-SRSS-TB
Changed lines of the file:
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@@
 		(property "Value" "100nF"
 			(at 73.914 112.9792 0)
-			(hide yes)
 			(show_name no)
 			(do_not_autoplace no)
@@
 		(property "ALTIUM_VALUE" "100nF(0402)"
 			(at 78.486 120.8532 0)
+			(hide yes)
 			(show_name no)
 			(do_not_autoplace no)
@@
 			(effects (font (size 1.27 1.27)))
 		)
-		(property "MPN" ""
+		(property "MPN" "SM02B-SRSS-TB"
 			(at 177.8 143.9672 0)
 			(hide yes)
@@
 			)
 		)
-		(property "Value" "JST_SH-02P"
+		(property "Value" "SM02B-SRSS-TB"
 			(at 172.72 154.1272 90)
 			(show_name no)
@@
 		(property "Value" "220pF"
 			(at 164.592 101.0412 90)
-			(hide yes)
 			(show_name no)
 			(do_not_autoplace no)
@@
 		(property "ALTIUM_VALUE" "560pF(0402)"
 			(at 167.386 108.1532 90)
+			(hide yes)
 			(show_name no)
 			(do_not_autoplace no)
@@
 		(property "Value" "100R"
 			(at 174.752 92.4052 90)
-			(hide yes)
 			(show_name no)
 			(do_not_autoplace no)
@@
 		(property "ALTIUM_VALUE" "100R(0402)"
 			(at 177.546 96.4692 90)
+			(hide yes)
 			(show_name no)
 			(do_not_autoplace no)
@@
 		(property "Value" "220pF"
 			(at 164.592 90.8812 90)
-			(hide yes)
 			(show_name no)
 			(do_not_autoplace no)
@@
 		(property "ALTIUM_VALUE" "560pF(0402)"
 			(at 167.386 97.9932 90)
+			(hide yes)
 			(show_name no)
 			(do_not_autoplace no)
@@
 		(property "Value" "100R"
 			(at 174.752 102.5652 90)
-			(hide yes)
 			(show_name no)
 			(do_not_autoplace no)
@@
 		(property "ALTIUM_VALUE" "100R(0402)"
 			(at 177.546 106.6292 90)
+			(hide yes)
 			(show_name no)
 			(do_not_autoplace no)
@@
 			(effects (font (size 1.27 1.27)))
 		)
-		(property "MPN" ""
+		(property "MPN" "SM02B-SRSS-TB"
 			(at 177.8 128.7272 0)
 			(hide yes)
@@
 			)
 		)
-		(property "Value" "JST_SH-02P"
+		(property "Value" "SM02B-SRSS-TB"
 			(at 172.72 138.8872 90)
 			(show_name no)
@@
 		(property "Value" "4k7"
 			(at 95.758 115.5192 0)
-			(hide yes)
 			(show_name no)
 			(do_not_autoplace no)
@@
 		(property "ALTIUM_VALUE" "4k7(0402)"
 			(at 97.282 123.3932 0)
-			(show_name no)
-			(do_not_autoplace no)
+			(hide yes)
+			(show_name no)
+			(do_not_autoplace no)
