File: STM32-FOC-hardware/ESC-BLDC/gate driver.kicad_sch (KiCad schematic)
At the start: 33 parts, among them J1 JUMPER, J2 JUMPER, U1 DRV8302DCA

Commit message: Use 4.7uF Basic capacitor for C10
Parts:
- C10: value 2.2uF -> 4.7uF; JLCPCB Class (none) -> Basic; LCSC C3870388 -> C23733; MPN (none) -> CL05A475MP5NRNC; Manufacturer (none) -> Samsung Electro-Mechanics
Changed lines of the file:
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@@
 		(in_pos_files yes)
 		(dnp no)
-		(property "LCSC" "C3870388"
+		(property "LCSC" "C23733"
 			(at 99.06 108.4072 0)
 			(hide yes)
@@
 				)
 			)
+		)
+		(property "Manufacturer" "Samsung Electro-Mechanics"
+			(at 99.06 108.4072 0)
+			(hide yes)
+			(show_name no)
+			(do_not_autoplace no)
+			(effects (font (size 1.27 1.27)))
+		)
+		(property "MPN" "CL05A475MP5NRNC"
+			(at 99.06 108.4072 0)
+			(hide yes)
+			(show_name no)
+			(do_not_autoplace no)
+			(effects (font (size 1.27 1.27)))
+		)
+		(property "JLCPCB Class" "Basic"
+			(at 99.06 108.4072 0)
+			(hide yes)
+			(show_name no)
+			(do_not_autoplace no)
+			(effects (font (size 1.27 1.27)))
 		)
 		(property "Reference" "C10"
@@
 			)
 		)
-		(property "Value" "2.2uF"
+		(property "Value" "4.7uF"
 			(at 96.774 107.8992 0)
 			(hide yes)
@@
 			)
 		)
-		(property "Description" "Chip capacitor, 2.2µF, 10%, 10V, 0402"
+		(property "Description" "4.7uF 10V X5R ±20% 0402 MLCC"
 			(at 99.06 108.4072 0)
 			(hide yes)

Commit message: Restore agreed L1 JLCPCB selection
Parts:
- L1: LCSC C6824612 -> C42462944
Changed lines of the file:
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@@
 		(in_pos_files yes)
 		(dnp no)
-		(property "LCSC" "C6824612"
+		(property "LCSC" "C42462944"
 			(at 220.98 90.6272 0)
 			(hide yes)

Commit message: Select stocked L1 inductor for assembly
Parts:
- L1: DC RESISTANCE (DCR) 135mR -> 98mR; DEPTH 6.72mm -> 6.6mm; LCSC C42462944 -> C22463831; LENGTH 7.24mm -> 7.1mm; MAX DC CURRENT 2.9A -> 3A; MPN ZEPI.0630A.220MT -> SL0650-220M; RMS CURRENT (IRMS) 2.9A -> 3A; SATURATION CURRENT 2.5A -> 5A
Changed lines of the file:
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@@
 		(in_pos_files yes)
 		(dnp no)
-		(property "LCSC" "C42462944"
+		(property "LCSC" "C22463831"
 			(at 220.98 90.6272 0)
 			(hide yes)
@@
 			(effects (font (size 1.27 1.27)))
 		)
-		(property "MPN" "ZEPI.0630A.220MT"
+		(property "MPN" "SL0650-220M"
 			(at 220.98 90.6272 0)
 			(hide yes)
@@
 			)
 		)
-		(property "Description" "Molded shielded inductor, 22uH, 3A rated, 3.5A saturation, 126mΩ, 7.1x6.6mm"
+		(property "Description" "Molded shielded inductor, 22uH, 3A rated, 5A saturation, 98mΩ, 7.1x6.6mm"
 			(at 220.98 90.6272 0)
 			(hide yes)
@@
 			)
 		)
-		(property "MAX DC CURRENT" "2.9A"
+		(property "MAX DC CURRENT" "3A"
 			(at 220.472 89.3572 90)
 			(hide yes)
@@
 			)
 		)
-		(property "DC RESISTANCE (DCR)" "135mR"
+		(property "DC RESISTANCE (DCR)" "98mR"
 			(at 220.472 89.3572 90)
 			(hide yes)
@@
 			)
 		)
-		(property "RMS CURRENT (IRMS)" "2.9A"
+		(property "RMS CURRENT (IRMS)" "3A"
 			(at 220.472 89.3572 90)
 			(hide yes)
@@
 			)
 		)
-		(property "SATURATION CURRENT" "2.5A"
-			(at 220.472 89.3572 90)
-			(hide yes)
-			(show_name no)
-			(do_not_autoplace no)
-			(effects
-				(font
-					(size 1.27 1.27)
-				)
-				(justify right bottom)
-			)
-		)
-		(property "LENGTH" "7.24mm"
-			(at 220.472 89.3572 90)
-			(hide yes)
-			(show_name no)
-			(do_not_autoplace no)
-			(effects
-				(font
-					(size 1.27 1.27)
-				)
-				(justify right bottom)
-			)
-		)
-		(property "DEPTH" "6.72mm"
-			(at 220.472 89.3572 90)
-			(hide yes)
+		(property "SATURATION CURRENT" "5A"
+			(at 220.472 89.3572 90)
+			(hide yes)
+			(show_name no)
+			(do_not_autoplace no)
+			(effects
+				(font
+					(size 1.27 1.27)
+				)
+				(justify right bottom)
+			)
+		)
+		(property "LENGTH" "7.1mm"
+			(at 220.472 89.3572 90)
+			(hide yes)
+			(show_name no)
+			(do_not_autoplace no)
+			(effects
+				(font
+					(size 1.27 1.27)
+				)
+				(justify right bottom)
+			)
+		)
+		(property "DEPTH" "6.6mm"
+			(at 220.472 89.3572 90)
+			(hide yes)

Commit message: Apply schematic cleanup and sourcing todo
Changed lines of the file:
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@@
 		(property "Value" "JUMPER"
 			(at 77.47 96.9772 90)
-			(hide yes)
 			(show_name no)
 			(do_not_autoplace no)
@@
 		(property "ALTIUM_VALUE" ""
 			(at 77.978 98.2472 90)
+			(hide yes)
 			(show_name no)
 			(do_not_autoplace no)
@@
 		(property "Value" "47uF"
 			(at 236.474 95.1992 0)
-			(hide yes)
 			(show_name no)
 			(do_not_autoplace no)
@@
 		(property "ALTIUM_VALUE" "47µF"
 			(at 241.046 103.0732 0)
+			(hide yes)
 			(show_name no)
 			(do_not_autoplace no)
@@
 		(property "Value" "100nF"
 			(at 179.832 118.8212 90)
-			(hide yes)
 			(show_name no)
 			(do_not_autoplace no)
@@
 		(property "ALTIUM_VALUE" "100nF"
 			(at 177.8 123.6472 90)
+			(hide yes)
 			(show_name no)
 			(do_not_autoplace no)
@@
 		(property "Value" "100pF"
 			(at 109.474 46.9392 0)
-			(hide yes)
 			(show_name no)
 			(do_not_autoplace no)
@@
 		(property "ALTIUM_VALUE" "120pF"
 			(at 114.046 54.8132 0)
+			(hide yes)
 			(show_name no)
 			(do_not_autoplace no)
@@
 		(property "Value" "3k3"
 			(at 90.424 59.6392 0)
-			(hide yes)
 			(show_name no)
 			(do_not_autoplace no)
@@
 		(property "ALTIUM_VALUE" "3k3"
 			(at 92.456 67.5132 0)
+			(hide yes)
 			(show_name no)
 			(do_not_autoplace no)
@@
 		(property "Value" "1M"
 			(at 204.724 95.1992 0)
-			(hide yes)
 			(show_name no)
 			(do_not_autoplace no)
@@
 		(property "ALTIUM_VALUE" "1M"
 			(at 206.756 103.0732 0)
+			(hide yes)
 			(show_name no)
 			(do_not_autoplace no)
@@
 		(property "Value" "1uF"
 			(at 96.774 133.2992 0)
-			(hide yes)
 			(show_name no)
 			(do_not_autoplace no)
@@
 		(property "ALTIUM_VALUE" "1µF"
 			(at 101.346 141.1732 0)
+			(hide yes)
 			(show_name no)
 			(do_not_autoplace no)
@@
 		(property "Value" "4.7uF"
 			(at 198.374 151.0792 0)
-			(hide yes)
 			(show_name no)
 			(do_not_autoplace no)
@@
 		(property "ALTIUM_VALUE" "4.7µF"
 			(at 202.946 158.9532 0)
+			(hide yes)
 			(show_name no)
 			(do_not_autoplace no)
@@
 		(property "Value" "10nF"
 			(at 178.054 59.6392 0)
-			(hide yes)
 			(show_name no)
 			(do_not_autoplace no)
@@
 		(property "ALTIUM_VALUE" "15nF"
 			(at 182.626 67.5132 0)
+			(hide yes)
 			(show_name no)
 			(do_not_autoplace no)
@@
 		(property "Value" "100R"
 			(at 90.932 160.7312 90)
-			(hide yes)
 			(show_name no)
 			(do_not_autoplace no)
@@
 		(property "ALTIUM_VALUE" "56R"
 			(at 93.726 165.3032 90)
+			(hide yes)
 			(show_name no)
 			(do_not_autoplace no)
@@
 		(property "Value" "100nF"
 			(at 183.134 151.0792 0)
-			(hide yes)
 			(show_name no)
 			(do_not_autoplace no)
@@
 		(property "ALTIUM_VALUE" "100nF"
 			(at 187.706 158.9532 0)
+			(hide yes)
 			(show_name no)
 			(do_not_autoplace no)
@@
 		(property "Value" "4.7uF"
 			(at 205.994 59.6392 0)
-			(hide yes)
 			(show_name no)
 			(do_not_autoplace no)
@@
 		(property "ALTIUM_VALUE" "4.7µF"
 			(at 210.566 67.5132 0)
+			(hide yes)
 			(show_name no)
 			(do_not_autoplace no)
@@
 		(property "Value" "JUMPER"
 			(at 77.47 107.1372 90)
-			(hide yes)
 			(show_name no)
 			(do_not_autoplace no)
@@
 		(property "ALTIUM_VALUE" ""
 			(at 77.978 108.4072 90)
+			(hide yes)
 			(show_name no)
 			(do_not_autoplace no)
@@
 		(property "Value" "1nF"
 			(at 86.614 163.7792 0)
-			(hide yes)
 			(show_name no)
 			(do_not_autoplace no)
@@
 		(property "ALTIUM_VALUE" "2.2nF"
 			(at 91.186 171.6532 0)
+			(hide yes)
 			(show_name no)
 			(do_not_autoplace no)
@@
 		(property "Value" "100nF"
 			(at 179.832 106.1212 90)
-			(hide yes)
 			(show_name no)
 			(do_not_autoplace no)
@@
 		(property "ALTIUM_VALUE" "100nF"
 			(at 177.8 110.9472 90)
+			(hide yes)
 			(show_name no)
 			(do_not_autoplace no)
@@
 		(property "Value" "100nF"
 			(at 192.532 83.2612 90)
-			(hide yes)
 			(show_name no)
 			(do_not_autoplace no)
@@
 		(property "ALTIUM_VALUE" "100nF"
 			(at 195.326 90.3732 90)
+			(hide yes)
 			(show_name no)
 			(do_not_autoplace no)
@@
 		(property "Value" "100R"
 			(at 90.932 153.1112 90)
-			(hide yes)
 			(show_name no)
 			(do_not_autoplace no)
@@
 		(property "ALTIUM_VALUE" "56R"
 			(at 93.726 157.6832 90)
+			(hide yes)
 			(show_name no)
 			(do_not_autoplace no)
@@
 		(property "Value" "100nF"
 			(at 193.294 59.6392 0)
-			(hide yes)
 			(show_name no)
 			(do_not_autoplace no)
@@
 		(property "ALTIUM_VALUE" "100nF"
 			(at 197.866 67.5132 0)
+			(hide yes)
 			(show_name no)
 			(do_not_autoplace no)
@@
 		(property "Value" "1k"
 			(at 77.724 128.2192 0)
-			(hide yes)
 			(show_name no)
 			(do_not_autoplace no)
@@
 		(property "ALTIUM_VALUE" "RB"
 			(at 79.756 136.0932 0)
+			(hide yes)
 			(show_name no)
 			(do_not_autoplace no)
@@
 		(property "Value" "15k"
 			(at 103.124 39.3192 0)
-			(hide yes)
 			(show_name no)
 			(do_not_autoplace no)
@@
 		(property "ALTIUM_VALUE" "15k"
 			(at 105.156 47.1932 0)
+			(hide yes)
 			(show_name no)
 			(do_not_autoplace no)
@@
 		(property "Value" "4.7uF"
 			(at 96.774 107.8992 0)
-			(hide yes)
 			(show_name no)
 			(do_not_autoplace no)
@@
 		(property "ALTIUM_VALUE" "2.2µF"
 			(at 101.346 115.7732 0)
+			(hide yes)
 			(show_name no)
 			(do_not_autoplace no)
@@
 		(property "Value" "18k"
 			(at 90.424 44.3992 0)
-			(hide yes)
 			(show_name no)
 			(do_not_autoplace no)
@@
 		(property "ALTIUM_VALUE" "18k"
 			(at 92.456 52.2732 0)
+			(hide yes)
 			(show_name no)
 			(do_not_autoplace no)
@@
 		(property "Value" "22nF"
 			(at 106.934 107.8992 0)
-			(hide yes)
 			(show_name no)
 			(do_not_autoplace no)
@@
 		(property "ALTIUM_VALUE" "22nF"
 			(at 111.506 115.7732 0)
+			(hide yes)
 			(show_name no)
 			(do_not_autoplace no)
@@
 		(property "Value" "1nF"
 			(at 76.454 163.7792 0)
-			(hide yes)
 			(show_name no)
 			(do_not_autoplace no)
@@
 		(property "ALTIUM_VALUE" "2.2nF"
 			(at 81.026 171.6532 0)
+			(hide yes)
 			(show_name no)
 			(do_not_autoplace no)
@@
 		(property "Value" "12k"
 			(at 103.632 89.6112 90)
-			(hide yes)
 			(show_name no)
 			(do_not_autoplace no)
@@
 		(property "ALTIUM_VALUE" "10k"
 			(at 106.426 94.1832 90)
+			(hide yes)
 			(show_name no)
 			(do_not_autoplace no)
@@
 		(property "Value" "10nF"
 			(at 101.854 54.5592 0)
-			(hide yes)
 			(show_name no)
 			(do_not_autoplace no)
@@
 		(property "ALTIUM_VALUE" "6.8nF"
 			(at 106.426 62.4332 0)
+			(hide yes)
 			(show_name no)
 			(do_not_autoplace no)
@@
 		(property "Value" "100nF"
 			(at 179.832 93.4212 90)
-			(hide yes)
 			(show_name no)
 			(do_not_autoplace no)
@@
 		(property "ALTIUM_VALUE" "100nF"
 			(at 177.8 98.2472 90)
+			(hide yes)
 			(show_name no)
 			(do_not_autoplace no)
@@
 		(property "Value" "39k"
 			(at 77.724 112.9792 0)
-			(hide yes)
 			(show_name no)
 			(do_not_autoplace no)
@@
 		(property "ALTIUM_VALUE" "RA"
 			(at 79.756 120.8532 0)
+			(hide yes)
 			(show_name no)
 			(do_not_autoplace no)
@@
 		(property "Value" "1uF"
 			(at 119.634 143.4592 0)
-			(hide yes)
 			(show_name no)
 			(do_not_autoplace no)
@@
 		(property "ALTIUM_VALUE" "1µF"
 			(at 124.206 151.3332 0)
+			(hide yes)
 			(show_name no)
 			(do_not_autoplace no)
@@
 		(property "Value" "200k"
 			(at 128.524 49.4792 0)
-			(hide yes)
 			(show_name no)
 			(do_not_autoplace no)
@@
 		(property "ALTIUM_VALUE" "200k"
 			(at 130.556 57.3532 0)
+			(hide yes)
 			(show_name no)
 			(do_not_autoplace no)
