File: STM32-FOC-hardware/ESC-BLDC/main controller.kicad_sch (KiCad schematic)
At the start: 21 parts, among them P10 HEADER-4P, P9 JST_SH-04P, U5 USBLC6-2SC6Y, U6 STM32F405RGT6, X1 12MHz

Commit message: Exclude unresolved JST connectors from assembly
Parts:
- P9: DNP (none) -> Yes; LCSC C160404 -> (none); MPN SM04B-SRSS-TB(LF)(SN) -> (none); now not fitted; now left out of the parts list
Changed lines of the file:
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@@
 		(body_style 1)
 		(exclude_from_sim no)
-		(in_bom yes)
+		(in_bom no)
 		(on_board yes)
-		(in_pos_files yes)
-		(dnp no)
-		(property "LCSC" "C160404"
+		(in_pos_files no)
+		(dnp yes)
+		(property "DNP" "Yes"
 			(at 175.26 60.1472 0)
 			(hide yes)
@@
 			(effects (font (size 1.27 1.27)))
 		)
-		(property "MPN" "SM04B-SRSS-TB(LF)(SN)"
+		(property "LCSC" ""
 			(at 175.26 60.1472 0)
 			(hide yes)
+			(show_name no)
+			(do_not_autoplace no)
+			(effects (font (size 1.27 1.27)))
+		)
+		(property "MPN" ""
+			(at 175.26 60.1472 0)
+			(hide yes)

Commit message: Apply schematic cleanup and sourcing todo
Parts:
- P9: value JST_SH-04P -> SM04B-SRSS-TB; MPN (none) -> SM04B-SRSS-TB
Changed lines of the file:
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@@
 		(property "Value" "12k"
 			(at 57.912 143.2052 90)
-			(hide yes)
 			(show_name no)
 			(do_not_autoplace no)
@@
 		(property "ALTIUM_VALUE" "12k(0402)"
 			(at 60.706 147.2692 90)
+			(hide yes)
 			(show_name no)
 			(do_not_autoplace no)
@@
 		(property "Value" "100nF"
 			(at 208.534 158.6992 0)
-			(hide yes)
 			(show_name no)
 			(do_not_autoplace no)
@@
 		(property "ALTIUM_VALUE" "100nF(0402)"
 			(at 213.106 166.5732 0)
+			(hide yes)
 			(show_name no)
 			(do_not_autoplace no)
@@
 		(property "Value" "100nF"
 			(at 190.754 158.6992 0)
-			(hide yes)
 			(show_name no)
 			(do_not_autoplace no)
@@
 		(property "ALTIUM_VALUE" "100nF(0402)"
 			(at 195.326 166.5732 0)
+			(hide yes)
 			(show_name no)
 			(do_not_autoplace no)
@@
 		(property "Value" "100R"
 			(at 96.012 46.6852 90)
-			(hide yes)
 			(show_name no)
 			(do_not_autoplace no)
@@
 		(property "ALTIUM_VALUE" "100R(0402)"
 			(at 98.806 50.7492 90)
+			(hide yes)
 			(show_name no)
 			(do_not_autoplace no)
@@
 		(property "Value" "100nF"
 			(at 112.014 133.2992 0)
-			(hide yes)
 			(show_name no)
 			(do_not_autoplace no)
@@
 		(property "ALTIUM_VALUE" "100nF(0402)"
 			(at 116.586 141.1732 0)
+			(hide yes)
 			(show_name no)
 			(do_not_autoplace no)
@@
 		(property "Value" "100nF"
 			(at 241.554 105.3592 0)
-			(hide yes)
 			(show_name no)
 			(do_not_autoplace no)
@@
 		(property "ALTIUM_VALUE" "100nF(0402)"
 			(at 246.126 113.2332 0)
+			(hide yes)
 			(show_name no)
 			(do_not_autoplace no)
@@
 		(property "Value" "100R"
 			(at 96.012 56.8452 90)
-			(hide yes)
 			(show_name no)
 			(do_not_autoplace no)
@@
 		(property "ALTIUM_VALUE" "100R(0402)"
 			(at 98.806 60.9092 90)
+			(hide yes)
 			(show_name no)
 			(do_not_autoplace no)
@@
 		(property "Value" "100nF"
 			(at 188.214 31.6992 0)
-			(hide yes)
 			(show_name no)
 			(do_not_autoplace no)
@@
 		(property "ALTIUM_VALUE" "100nF(0402)"
 			(at 192.786 39.5732 0)
+			(hide yes)
 			(show_name no)
 			(do_not_autoplace no)
@@
 		(property "Value" "100nF"
 			(at 223.774 105.3592 0)
-			(hide yes)
 			(show_name no)
 			(do_not_autoplace no)
@@
 		(property "ALTIUM_VALUE" "100nF(0402)"
 			(at 228.346 113.2332 0)
+			(hide yes)
 			(show_name no)
 			(do_not_autoplace no)
@@
 			(effects (font (size 1.27 1.27)))
 		)
-		(property "MPN" ""
+		(property "MPN" "SM04B-SRSS-TB"
 			(at 175.26 60.1472 0)
 			(hide yes)
@@
 			)
 		)
-		(property "Value" "JST_SH-04P"
+		(property "Value" "SM04B-SRSS-TB"
 			(at 170.18 62.6872 90)
 			(show_name no)
@@
 		(property "Value" "1k"
 			(at 44.958 161.2392 0)
-			(hide yes)
 			(show_name no)
 			(do_not_autoplace no)
@@
 		(property "ALTIUM_VALUE" "1k(0402)"
 			(at 46.482 169.1132 0)
+			(hide yes)
 			(show_name no)
 			(do_not_autoplace no)
@@
 		(property "Value" "100nF"
 			(at 139.954 69.7992 0)
-			(hide yes)
 			(show_name no)
 			(do_not_autoplace no)
@@
 		(property "ALTIUM_VALUE" "100nF(0402)"
 			(at 144.526 77.6732 0)
+			(hide yes)
 			(show_name no)
 			(do_not_autoplace no)
@@
 		(property "Value" "12k"
 			(at 57.912 135.5852 90)
-			(hide yes)
 			(show_name no)
 			(do_not_autoplace no)
@@
 		(property "ALTIUM_VALUE" "12k(0402)"
 			(at 60.706 139.6492 90)
+			(hide yes)
 			(show_name no)
 			(do_not_autoplace no)
@@
 		(property "Value" "100nF"
 			(at 142.494 171.3992 0)
-			(hide yes)
 			(show_name no)
 			(do_not_autoplace no)
@@
 		(property "ALTIUM_VALUE" "100nF(0402)"
 			(at 147.066 179.2732 0)
+			(hide yes)
 			(show_name no)
 			(do_not_autoplace no)
