File: STM32-FOC-hardware/ESC-BLDC/rotor angle sensor.kicad_sch (KiCad schematic)
At the start: 7 parts, among them P6 JST_SH-05P, U3 AS5047P

Commit message: Exclude unresolved JST connectors from assembly
Parts:
- P6: DNP (none) -> Yes; LCSC C136657 -> (none); MPN SM05B-SRSS-TB(LF)(SN) -> (none); now not fitted; now left out of the parts list
Changed lines of the file:
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@@
 		(body_style 1)
 		(exclude_from_sim no)
-		(in_bom yes)
+		(in_bom no)
 		(on_board yes)
-		(in_pos_files yes)
-		(dnp no)
-		(property "LCSC" "C136657"
+		(in_pos_files no)
+		(dnp yes)
+		(property "DNP" "Yes"
 			(at 53.34 121.1072 0)
 			(hide yes)
@@
 			(effects (font (size 1.27 1.27)))
 		)
-		(property "MPN" "SM05B-SRSS-TB(LF)(SN)"
+		(property "LCSC" ""
 			(at 53.34 121.1072 0)
 			(hide yes)
+			(show_name no)
+			(do_not_autoplace no)
+			(effects (font (size 1.27 1.27)))
+		)
+		(property "MPN" ""
+			(at 53.34 121.1072 0)
+			(hide yes)

Commit message: Apply schematic cleanup and sourcing todo
Parts:
- P6: value JST_SH-05P -> SM05B-SRSS-TB; MPN (none) -> SM05B-SRSS-TB
- R28, R29: DNP (none) -> Yes; now not fitted; now left out of the parts list
Changed lines of the file:
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@@
 		(body_style 1)
 		(exclude_from_sim no)
-		(in_bom yes)
+		(in_bom no)
 		(on_board yes)
-		(in_pos_files yes)
-		(dnp no)
+		(in_pos_files no)
+		(dnp yes)
+		(property "DNP" "Yes"
+			(at 68.58 116.0272 0)
+			(hide yes)
+			(show_name no)
+			(do_not_autoplace no)
+			(effects (font (size 1.27 1.27)))
+		)
 		(property "Reference" "R29"
 			(at 73.66 116.0272 90)
@@
 		(property "Value" "0R"
 			(at 67.31 119.8372 90)
-			(hide yes)
 			(show_name no)
 			(do_not_autoplace no)
@@
 		(property "ALTIUM_VALUE" "0R(0402)"
 			(at 60.96 116.0272 90)
+			(hide yes)
 			(show_name no)
 			(do_not_autoplace no)
@@
 		(property "Value" "0R"
 			(at 67.31 122.3772 90)
-			(hide yes)
 			(show_name no)
 			(do_not_autoplace no)
@@
 		(property "ALTIUM_VALUE" "0R(0402)"
 			(at 60.96 118.5672 90)
+			(hide yes)
 			(show_name no)
 			(do_not_autoplace no)
@@
 		(property "Value" "100nF"
 			(at 203.454 107.8992 0)
-			(hide yes)
 			(show_name no)
 			(do_not_autoplace no)
@@
 		(property "ALTIUM_VALUE" "100nF(0402)"
 			(at 208.026 115.7732 0)
+			(hide yes)
 			(show_name no)
 			(do_not_autoplace no)
@@
 			(effects (font (size 1.27 1.27)))
 		)
-		(property "MPN" ""
+		(property "MPN" "SM05B-SRSS-TB"
 			(at 53.34 121.1072 0)
 			(hide yes)
@@
 			)
 		)
-		(property "Value" "JST_SH-05P"
+		(property "Value" "SM05B-SRSS-TB"
 			(at 48.26 123.6472 90)
 			(show_name no)
@@
 		(body_style 1)
 		(exclude_from_sim no)
-		(in_bom yes)
+		(in_bom no)
 		(on_board yes)
-		(in_pos_files yes)
-		(dnp no)
+		(in_pos_files no)
+		(dnp yes)
+		(property "DNP" "Yes"
+			(at 68.58 113.4872 0)
+			(hide yes)
+			(show_name no)
+			(do_not_autoplace no)
+			(effects (font (size 1.27 1.27)))
+		)
 		(property "Reference" "R28"
 			(at 73.66 113.4872 90)
@@
 		(property "Value" "0R"
 			(at 67.31 117.2972 90)
-			(hide yes)
 			(show_name no)
 			(do_not_autoplace no)
@@
 		(property "ALTIUM_VALUE" "0R(0402)"
 			(at 60.96 113.4872 90)
+			(hide yes)
 			(show_name no)
 			(do_not_autoplace no)
@@
 		(property "Value" "100nF"
 			(at 66.294 90.1192 0)
-			(hide yes)
 			(show_name no)
 			(do_not_autoplace no)
@@
 		(property "ALTIUM_VALUE" "100nF(0402)"
 			(at 70.866 97.9932 0)
-			(show_name no)
-			(do_not_autoplace no)
+			(hide yes)
+			(show_name no)
+			(do_not_autoplace no)
